File: CC2650_with_Discrete_v1.0/CC2650_with_Discrete.sch (KiCad schematic (older format))
At the start: 70 parts, among them J1 SMA_EDGE_CONNECTOR, P1 CONN_02X03, P2 JTAG, P3 XBEE, SW1 RESET, SW2 USER_BUTTON, U1 TPS63051, U2 cc2650_7x7, U3 LTR-303ALS, U4 Si7006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

Commit message: verified schematic; added reference
- verified schematic for both discrete and balun
- added reference datasheet
- removed library directory
Parts:
- removed J1: SMA_EDGE_CONNECTOR, symbol SMA_10V21_TGG
- removed P1: CONN_02X03, Socket_Strips:Socket_Strip_Angled_2x03, symbol CONN_02X03
- added P1: CONN_02X04, symbol CONN_02X04
- added U5: EDGE_SMA, symbol EDGE_SMA
Connections:
- wire segments 241 -> 243
Changed lines of the file:
@@
 EESchema Schematic File Version 2
-LIBS:CC2650_with_Discrete-rescue
 LIBS:power
 LIBS:device
@@
 LIBS:si7006
 LIBS:ltr-303als
-LIBS:sma_10v21_tgg
 LIBS:crystal_24MHz
 LIBS:inductor
 LIBS:tps63051
 LIBS:tps782
+LIBS:JTAG
 LIBS:cc2650_7x7
-LIBS:JTAG
+LIBS:antenna_2.4GHz
+LIBS:edge_sma
 EELAYER 25 0
 EELAYER END
@@
 $EndComp
 $Comp
-L SMA_10V21_TGG J1
-U 1 1 58331F13
-P 10075 4550
-F 0 "J1" H 10125 4400 60  0000 C CNN
-F 1 "SMA_EDGE_CONNECTOR" H 10075 4750 60  0000 C CNN
-F 2 "" H 10075 4550 60  0001 C CNN
-F 3 "" H 10075 4550 60  0001 C CNN
-	1    10075 4550
-	1    0    0    -1
-$EndComp
-$Comp
 L Si7006 U4
 U 1 1 5835C02D
@@
 Text GLabel 4300 4725 1    39   Input ~ 0
 INTR
-$Comp
-L CONN_02X03 P1
-U 1 1 5845B71F
-P 7575 9800
-F 0 "P1" H 7575 10000 50  0000 C CNN
-F 1 "CONN_02X03" H 7575 9600 50  0000 C CNN
-F 2 "Socket_Strips:Socket_Strip_Angled_2x03" H 7575 8600 50  0001 C CNN
-F 3 "" H 7575 8600 50  0000 C CNN
-	1    7575 9800
-	1    0    0    -1
-$EndComp
 Text GLabel 7200 9700 0    39   Input ~ 0
 DIO_1
@@
 Wire Wire Line
 	8950 5425 8950 5375
+$Comp
+L CONN_02X04 P1
+U 1 1 5844BD1F
+P 7575 9750
+F 0 "P1" H 7575 10000 50  0000 C CNN
+F 1 "CONN_02X04" H 7575 9500 50  0000 C CNN
+F 2 "" H 7575 8550 50  0000 C CNN
+F 3 "" H 7575 8550 50  0000 C CNN
+	1    7575 9750
+	1    0    0    -1
+$EndComp
+Text GLabel 7200 9600 0    39   Input ~ 0
+VDDS
+Wire Wire Line
+	7200 9600 7325 9600
+$Comp
+L EDGE_SMA U5
+U 1 1 5845D8F7
+P 10075 4550
+F 0 "U5" H 10125 4400 60  0000 C CNN
+F 1 "EDGE_SMA" H 10075 4750 60  0000 C CNN
+F 2 "" H 10075 4550 60  0001 C CNN
+F 3 "" H 10075 4550 60  0001 C CNN
+	1    10075 4550
+	1    0    0    -1
+$EndComp
+Text GLabel 7950 9600 2    39   Input ~ 0
+DIO_0
+Wire Wire Line
+	7950 9600 7825 9600
 $EndSCHEMATC

Commit message: added schematic pdf
Parts:
- P3: symbol XBEE -> XBEE-RESCUE-CC2650_with_Discrete
Changed lines of the file:
@@
 EESchema Schematic File Version 2
+LIBS:CC2650_with_Discrete-rescue
 LIBS:power
 LIBS:device
@@
 LIBS:antenna_2.4GHz
 LIBS:edge_sma
+LIBS:CC2650_with_Discrete-cache
 EELAYER 25 0
 EELAYER END
@@
 Connector Section
 $Comp
-L XBEE P3
+L XBEE-RESCUE-CC2650_with_Discrete P3
 U 1 1 583976FC
 P 14200 8900
