File: CC2650_with_Balun_v1.0/CC2650_with_balun.sch (KiCad schematic (older format))
At the start: 65 parts, among them P1 CONN_02X03, P2 JTAG, P3 XBEE, SW1 RESET, SW2 USER_BUTTON, U1 TPS63051, U2 cc2650_7x7, U3 LTR-303ALS, U4 Si7006, U5 SMA_EDGE_CONNECTOR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

Commit message: verified schematic; added reference
- verified schematic for both discrete and balun
- added reference datasheet
- removed library directory
Parts:
- removed C29: 100pF, symbol C
- removed C30, C32: DNM, symbol C
- removed FL2: LFB182G45BG5D920, symbol LFB182G45BG5D920
- removed P1: CONN_02X03, symbol CONN_02X03
- removed U5: SMA_EDGE_CONNECTOR, symbol SMA_10V21_TGG
- added P1: CONN_02X04, symbol CONN_02X04
- added U5: 2450BM14G0011, symbol 2450BM14G0011
- added U7: EDGE_SMA, symbol EDGE_SMA
- Y2: value 24MHz -> 24 MHz
Connections:
- wire segments 234 -> 230

Commit message: added schematic pdf
Parts:
- P3: symbol XBEE -> XBEE-RESCUE-CC2650_with_balun
Changed lines of the file:
@@
 EESchema Schematic File Version 2
+LIBS:CC2650_with_balun-rescue
 LIBS:power
 LIBS:device
@@
 Connector Section
 $Comp
-L XBEE P3
+L XBEE-RESCUE-CC2650_with_balun P3
 U 1 1 583976FC
 P 14200 8900

Commit message: Updated README
Parts:
- removed C22: NC, symbol C
- C17, C25: value 22uF -> 10uF
- C20: value 100uF -> 100nF
- L6: value 6.8uH -> 10uH
Connections:
- net labels added: CC2650_VIN
- wire segments 230 -> 229
Other:
- note added: "PIN 13\n"
- note added: "PIN 22\n"
- note added: "PIN 34\n"
- note added: "PIN 44\n"
- note added: "Pin 45"
- note added: "Pin 48"
Changed lines of the file:
@@
 EESchema Schematic File Version 2
-LIBS:CC2650_with_balun-rescue
 LIBS:power
 LIBS:device
@@
 P 6700 2250
 F 0 "C17" H 6725 2350 50  0000 L CNN
-F 1 "22uF" H 6725 2150 50  0000 L CNN
+F 1 "10uF" H 6725 2150 50  0000 L CNN
 F 2 "" H 6738 2100 50  0000 C CNN
 F 3 "" H 6700 2250 50  0000 C CNN
@@
 P 7100 2250
 F 0 "C20" H 7125 2350 50  0000 L CNN
-F 1 "100uF" H 7125 2150 50  0000 L CNN
+F 1 "100nF" H 7125 2150 50  0000 L CNN
 F 2 "" H 7138 2100 50  0000 C CNN
 F 3 "" H 7100 2250 50  0000 C CNN
 	1    7100 2250
-	1    0    0    -1
-$EndComp
-$Comp
-L C C22
-U 1 1 582D9BB4
-P 7500 2250
-F 0 "C22" H 7525 2350 50  0000 L CNN
-F 1 "NC" H 7525 2150 50  0000 L CNN
-F 2 "" H 7538 2100 50  0000 C CNN
-F 3 "" H 7500 2250 50  0000 C CNN
-	1    7500 2250
 	1    0    0    -1
 $EndComp
@@
 P 9050 2250
 F 0 "C25" H 9075 2350 50  0000 L CNN
-F 1 "22uF" H 9075 2150 50  0000 L CNN
+F 1 "10uF" H 9075 2150 50  0000 L CNN
 F 2 "" H 9088 2100 50  0000 C CNN
 F 3 "" H 9050 2250 50  0000 C CNN
@@
 P 8550 2100
 F 0 "L6" V 8700 2100 50  0000 C CNN
-F 1 "6.8uH" V 8450 2100 50  0000 C CNN
+F 1 "10uH" V 8450 2100 50  0000 C CNN
 F 2 "" H 8550 2100 50  0000 C CNN
 F 3 "" H 8550 2100 50  0000 C CNN
@@
 $EndComp
 Text GLabel 3950 1600 1    39   Input ~ 0
-CC1310_VIN
+CC2650_VIN
 $Comp
 L R R8
@@
 $EndComp
 $Comp
-L GND #PWR25
-U 1 1 583CCECC
-P 7500 2525
-F 0 "#PWR25" H 7500 2275 50  0001 C CNN
-F 1 "GND" H 7500 2375 50  0000 C CNN
-F 2 "" H 7500 2525 50  0000 C CNN
-F 3 "" H 7500 2525 50  0000 C CNN
-	1    7500 2525
-	1    0    0    -1
-$EndComp
-$Comp
 L GND #PWR23
 U 1 1 583CD51D
@@
 Connection ~ 5000 2100
 Wire Wire Line
-	4750 2100 7500 2100
-Wire Wire Line
 	5200 6375 5450 6375
 Wire Wire Line
@@
 	10550 2500 10550 2400
 Wire Wire Line
-	7500 2525 7500 2400
-Wire Wire Line
 	2725 2075 2500 2075
 Wire Notes Line
@@
 	8025 5725 7900 5725
 Connection ~ 7900 5725
+Wire Wire Line
+	4750 2100 7100 2100
+Text Notes 5250 2075 0    60   ~ 0
+PIN 13\n
+Text Notes 5675 2075 0    60   ~ 0
+PIN 22\n
+Text Notes 6125 2075 0    60   ~ 0
+PIN 44\n
+Text Notes 6925 2075 0    60   ~ 0
+PIN 34\n
+Text Notes 9425 2075 0    60   ~ 0
+Pin 45
+Text Notes 10150 2075 0    60   ~ 0
+Pin 48
 $EndSCHEMATC
